Commit message: chore: changed the parameters for f1tenth xacro model

File: urdf/f1tenth.urdf.xacro (robot description, xacro)
@@ -1,10 +1,25 @@
 <?xml version="1.0"?>
 <!--
-This URDF description of the car is taken from the f1tenth_ros_gym package. Modifications
-are documented within the xml below.
+  URDF for F1Tenth Gazebo simulation.
+    - body_mass:  18.0 kg  → 3.5 kg   (realistic 1/10 scale car weight)
+    - wheel_mass: 0.5 kg   → 0.1 kg   (realistic RC tire weight)
+    - hinge_mass: 0.5 kg   → 0.1 kg   (lightweight steering knuckle)
+    - Body inertia recalculated for 3.5 kg solid box
+    - Wheel inertia recalculated for 0.1 kg cylinder
+    - Steering hinge limits: ±0.5 rad → ±0.31 rad (from VESC servo clamp)
+    - Steering hinge velocity: 5.0 → 3.2 rad/s (from throttle_interpolator max_servo_speed)
+    - Tire friction: mu1 1.5→0.8, mu2 2.5→1.0 (indoor smooth surface)
+    - Contact stiffness: kp 500000→100000 (less rigid tire contact)
+    - Laser position: 0.275→0.27 m (matches static_transform_publisher in launch)
+    - max_steer: 0.5→0.31 rad (matches VESC-derived steering limit)
+    - max_wheel_torque: 100→20 Nm (matches 2.5 m/s² accel limit at 3.5 kg)
+    - Steering PID: reduced for lighter mass to prevent overshoot
+    - Velocity PID: reduced for lighter mass
 -->
-<!-- A simple model of the racecar for rviz -->
 <robot xmlns:xacro="http://www.ros.org/wiki/xacro" name="racecar">
-  <xacro:property name="wheelbase" value="0.3302" />
+  <!-- ================================================================== -->
+  <!-- Geometric properties                                                -->
+  <!-- ================================================================== -->
+  <xacro:property name="wheelbase" value="0.25" />
   <xacro:property name="width" value="0.2032" />
   <xacro:property name="height" value="0.1" />
@@ -12,19 +27,40 @@
   <xacro:property name="wheel_radius" value="0.0508" />
   <xacro:property name="wheel_length" value="0.0381" />
-  <xacro:property name="laser_distance_from_base_link" value="0.275" />
+  <xacro:property name="car_name" value="ego_racecar" />
+  <!-- laser position from static_transform_publisher: 0.27m forward, 0.11m up -->
+  <xacro:property name="laser_distance_from_base_link" value="0.27" />
   <xacro:property name="laser_height" value="0.05" />
   <xacro:property name="laser_radius" value="0.026" />
-  <xacro:property name="car_name" value="ego_racecar" />
-  <!-- Mass properties -->
-  <xacro:property name="body_mass" value="18.0" />
-  <xacro:property name="wheel_mass" value="0.5" />
-  <xacro:property name="hinge_mass" value="0.5" />
-  <!-- Body inertia: solid box (wheelbase x width x height) at 18kg
-       ixx = (1/12)*m*(w^2+h^2) = 1.5*(0.04129+0.01)       = 0.0769
-       iyy = (1/12)*m*(l^2+h^2) = 1.5*(0.10903+0.01)       = 0.1786
-       izz = (1/12)*m*(l^2+w^2) = 1.5*(0.10903+0.04129)    = 0.2255  -->
-  <!-- Wheel inertia: solid cylinder (r=0.0508, h=0.0381) at 0.5kg
-       ixx = iyy = (1/12)*m*(3r^2+h^2) = 0.0417*(0.00774+0.00145) = 0.000383
-       izz = (1/2)*m*r^2 = 0.25*0.002581                           = 0.000645  -->
+  <!-- ================================================================== -->
+  <!-- Mass properties                                                     -->
+  <!--   Real F1Tenth car: ~3.2-3.8 kg total (chassis + battery + compute  -->
+  <!--   + LiDAR + VESC). Using 3.5 kg as body mass.                      -->
+  <!--   RC tires: ~80-120g each. Using 0.1 kg.                           -->
+  <!-- ================================================================== -->
+  <xacro:property name="body_mass" value="3.5" />
+  <xacro:property name="wheel_mass" value="0.1" />
+  <xacro:property name="hinge_mass" value="0.1" />
+  <!-- Steering limits derived from VESC config                 -->
+  <!--   servo range [0.15, 0.85], gain=-1.2135, offset=0.5304            -->
+  <!--   max angle = (0.85 - 0.5304) / 1.2135 ≈ 0.264 rad               -->
+  <!--   min angle = (0.15 - 0.5304) / 1.2135 ≈ -0.314 rad              -->
+  <!--   Using ±0.31 as symmetric approximation                           -->
+  <xacro:property name="max_steering_angle" value="0.31" />
+  <!-- Steering velocity from throttle_interpolator config      -->
+  <xacro:property name="max_steering_velocity" value="3.2" />
+  <!-- ================================================================== -->
+  <!-- Body inertia at 3.5 kg (solid box: 0.25 x 0.2032 x 0.1)-->
+  <!--   ixx = (1/12)*3.5*(0.2032² + 0.1²)  = 0.0150                     -->
+  <!--   iyy = (1/12)*3.5*(0.25²   + 0.1²)  = 0.0347                     -->
+  <!--   izz = (1/12)*3.5*(0.25²   + 0.2032²)= 0.0439                    -->
+  <!-- ================================================================== -->
+  <!-- ================================================================== -->
+  <!-- Wheel inertia at 0.1 kg (cylinder r=0.0508, h=0.0381)   -->
+  <!--   ixx = iyy = (1/12)*0.1*(3*0.0508² + 0.0381²) = 0.0000766        -->
+  <!--   izz = (1/2)*0.1*0.0508²                       = 0.000129         -->
+  <!-- ================================================================== -->
+  <!-- ================================================================== -->
+  <!-- Materials                                                           -->
+  <!-- ================================================================== -->
   <material name="black">
     <color rgba="0.2 0.2 0.2 1."/>
@@ -33,5 +69,7 @@
     <color rgba="0.3 0.57 1. 1."/>
   </material>
- <!-- Added collision and inertial tags to support Gazebo physics solver -->
+  <!-- ================================================================== -->
+  <!-- Base link (chassis)                                                 -->
+  <!-- ================================================================== -->
   <link name="${car_name}/base_link">
     <visual>
@@ -48,19 +86,23 @@
       </geometry>
     </collision>
+    <!-- mass and inertia for 3.5 kg -->
     <inertial>
       <origin xyz="${wheelbase/2} 0 ${ground_offset+height/2}"/>
       <mass value="${body_mass}"/>
-      <inertia ixx="0.0769" ixy="0.0" ixz="0.0"
-               iyy="0.1786" iyz="0.0"
-               izz="0.2255"/>
-    </inertial>
-  </link>
-  <!-- Render color for base link on Gazebo -->
+      <inertia ixx="0.0150" ixy="0.0" ixz="0.0"
+               iyy="0.0347" iyz="0.0"
+               izz="0.0439"/>
+    </inertial>
+  </link>
   <gazebo reference="${car_name}/base_link">
     <material>Gazebo/Blue</material>
   </gazebo>
+  <!-- ================================================================== -->
+  <!-- LiDAR (Hokuyo URG)                                                 -->
+  <!-- ================================================================== -->
   <joint name="base_to_laser_model" type="fixed">
     <parent link="${car_name}/base_link"/>
     <child link="${car_name}/laser_model"/>
+    <!-- x=0.27 to match static_transform_publisher in launch file -->
     <origin xyz="${laser_distance_from_base_link} 0 ${ground_offset+height+(laser_height/2)}"/>
   </joint>
@@ -73,5 +115,7 @@
     </visual>
   </link>
-  <!-- Continuous joint to allow wheel to rotate 360 degrees -->
+  <!-- ================================================================== -->
+  <!-- Back left wheel                                                     -->
+  <!-- ================================================================== -->
   <joint name="base_to_back_left_wheel" type="continuous">
     <parent link="${car_name}/base_link"/>
@@ -82,5 +126,4 @@
     <dynamics damping="0.01" friction="0.0"/>
   </joint>
-  <!-- Added collision and inertial tags to support Gazebo physics solver -->
   <link name="${car_name}/back_left_wheel">
     <visual>
@@ -97,22 +140,25 @@
       </geometry>
     </collision>
+    <!-- wheel inertia at 0.1 kg -->
     <inertial>
       <origin rpy="${pi/2} 0 0"/>
       <mass value="${wheel_mass}"/>
-      <inertia ixx="0.000383" ixy="0.0" ixz="0.0"
-               iyy="0.000383" iyz="0.0"
-               izz="0.000645"/>
-    </inertial>
-  </link>
-  <!-- Render color for back left wheel on Gazebo -->
+      <inertia ixx="0.0000766" ixy="0.0" ixz="0.0"
+               iyy="0.0000766" iyz="0.0"
+               izz="0.000129"/>
+    </inertial>
+  </link>
+  <!-- tire friction for indoor smooth surface -->
   <gazebo reference="${car_name}/back_left_wheel">
     <material>Gazebo/Black</material>
-    <mu1>1.5</mu1>
-    <mu2>2.5</mu2>
-    <kp>500000.0</kp>
+    <mu1>0.8</mu1>
+    <mu2>1.0</mu2>
+    <kp>100000.0</kp>
     <kd>10.0</kd>
     <minDepth>0.001</minDepth>
   </gazebo>
-  <!-- Continuous join to allow wheel to rotate 360 degrees -->
+  <!-- ================================================================== -->
+  <!-- Back right wheel                                                    -->
+  <!-- ================================================================== -->
   <joint name="base_to_back_right_wheel" type="continuous">
     <parent link="${car_name}/base_link"/>
@@ -123,5 +169,4 @@
     <dynamics damping="0.01" friction="0.0"/>
   </joint>
-  <!-- Added collision and inertial tags to support Gazebo physics solver -->
   <link name="${car_name}/back_right_wheel">
     <visual>
@@ -138,22 +183,26 @@
       </geometry>
     </collision>
+    <!-- wheel inertia at 0.1 kg -->
     <inertial>
       <origin rpy="${pi/2} 0 0"/>
       <mass value="${wheel_mass}"/>
-      <inertia ixx="0.000383" ixy="0.0" ixz="0.0"
-               iyy="0.000383" iyz="0.0"
-               izz="0.000645"/>
-    </inertial>
-  </link>
-  <!-- Render color for back right wheel on Gazebo -->
+      <inertia ixx="0.0000766" ixy="0.0" ixz="0.0"
+               iyy="0.0000766" iyz="0.0"
+               izz="0.000129"/>
+    </inertial>
+  </link>
+  <!-- tire friction for indoor smooth surface -->
   <gazebo reference="${car_name}/back_right_wheel">
     <material>Gazebo/Black</material>
-    <mu1>1.5</mu1>
-    <mu2>2.5</mu2>
-    <kp>500000.0</kp>
+    <mu1>0.8</mu1>
+    <mu2>1.0</mu2>
+    <kp>100000.0</kp>
     <kd>10.0</kd>
     <minDepth>0.001</minDepth>
   </gazebo>
-  <!-- Revolute joint to allow wheel axel to rotate along Z axis -->
+  <!-- ================================================================== -->
+  <!-- Front left steering hinge + wheel                                   -->
+  <!-- ================================================================== -->
+  <!-- steering limits from VESC servo config, velocity from throttle_interpolator -->
   <joint name="base_to_front_left_hinge" type="revolute">
     <parent link="${car_name}/base_link"/>
@@ -161,5 +210,5 @@
     <origin xyz="${wheelbase} ${(wheel_length+width)/2} ${wheel_radius}"/>
     <axis xyz="0 0 1"/>
-    <limit lower="-0.5" upper="0.5" effort="10.0" velocity="5.0"/>
+    <limit lower="-${max_steering_angle}" upper="${max_steering_angle}" effort="10.0" velocity="${max_steering_velocity}"/>
     <dynamics damping="0.1" friction="0.0"/>
   </joint>
@@ -172,5 +221,4 @@
     </inertial>
   </link>
-  <!-- Continuous joint to allow wheel to rotate 360 degrees -->
   <joint name="front_left_hinge_to_wheel" type="continuous">
     <parent link="${car_name}/front_left_hinge"/>
@@ -180,5 +228,4 @@
     <dynamics damping="0.01" friction="0.0"/>
   </joint>
-  <!-- Added collision and inertial tags to support Gazebo physics solver -->
   <link name="${car_name}/front_left_wheel">
     <visual>
@@ -195,22 +242,26 @@
       </geometry>
     </collision>
+    <!-- wheel inertia at 0.1 kg -->
     <inertial>
       <origin rpy="${pi/2} 0 0"/>
       <mass value="${wheel_mass}"/>
-      <inertia ixx="0.000383" ixy="0.0" ixz="0.0"
-               iyy="0.000383" iyz="0.0"
-               izz="0.000645"/>
-    </inertial>
-  </link>
-  <!-- Render color for front left wheel on Gazebo -->
+      <inertia ixx="0.0000766" ixy="0.0" ixz="0.0"
+               iyy="0.0000766" iyz="0.0"
+               izz="0.000129"/>
+    </inertial>
+  </link>
+  <!-- tire friction for indoor smooth surface -->
   <gazebo reference="${car_name}/front_left_wheel">
     <material>Gazebo/Black</material>
-    <mu1>1.5</mu1>
-    <mu2>2.5</mu2>
-    <kp>500000.0</kp>
+    <mu1>0.8</mu1>
+    <mu2>1.0</mu2>
+    <kp>100000.0</kp>
     <kd>10.0</kd>
     <minDepth>0.001</minDepth>
   </gazebo>
-  <!-- Revolute joint to allow wheel to spin 360 degrees -->
+  <!-- ================================================================== -->
+  <!-- Front right steering hinge + wheel                                  -->
+  <!-- ================================================================== -->
+  <!-- steering limits from VESC servo config, velocity from throttle_interpolator -->
   <joint name="base_to_front_right_hinge" type="revolute">
     <parent link="${car_name}/base_link"/>
@@ -218,5 +269,5 @@
     <origin xyz="${wheelbase} ${-(wheel_length+width)/2} ${wheel_radius}"/>
     <axis xyz="0 0 1"/>
-    <limit lower="-0.5" upper="0.5" effort="10.0" velocity="5.0"/>
+    <limit lower="-${max_steering_angle}" upper="${max_steering_angle}" effort="10.0" velocity="${max_steering_velocity}"/>
     <dynamics damping="0.1" friction="0.0"/>
   </joint>
@@ -229,5 +280,4 @@
     </inertial>
   </link>
-  <!-- Continuous joint to allow wheel to rotate 360 degrees -->
   <joint name="front_right_hinge_to_wheel" type="continuous">
     <parent link="${car_name}/front_right_hinge"/>
@@ -237,5 +287,4 @@
     <dynamics damping="0.01" friction="0.0"/>
   </joint>
-  <!-- Added collision and inertial tags to support Gazebo physics solver -->
   <link name="${car_name}/front_right_wheel">
     <visual>
@@ -252,23 +301,27 @@
       </geometry>
     </collision>
+    <!-- wheel inertia at 0.1 kg -->
     <inertial>
       <origin rpy="${pi/2} 0 0"/>
       <mass value="${wheel_mass}"/>
-      <inertia ixx="0.000383" ixy="0.0" ixz="0.0"
-               iyy="0.000383" iyz="0.0"
-               izz="0.000645"/>
-    </inertial>
-  </link>
-  <!-- Render color for front right wheel on Gazebo -->
+      <inertia ixx="0.0000766" ixy="0.0" ixz="0.0"
+               iyy="0.0000766" iyz="0.0"
+               izz="0.000129"/>
+    </inertial>
+  </link>
+  <!-- tire friction for indoor smooth surface -->
   <gazebo reference="${car_name}/front_right_wheel">
     <material>Gazebo/Black</material>
-    <mu1>1.5</mu1>
-    <mu2>2.5</mu2>
-    <kp>500000.0</kp>
+    <mu1>0.6</mu1>
+    <mu2>0.8</mu2>
+    <kp>100000.0</kp>
     <kd>10.0</kd>
     <minDepth>0.001</minDepth>
   </gazebo>
-  <!-- Include URDF description for camera -->
+  <!-- ================================================================== -->
+  <!-- Intel RealSense D435i Camera                                        -->
+  <!-- ================================================================== -->
   <xacro:include filename="$(find realsense2_description)/urdf/_d435i.urdf.xacro" />
+  <!-- TODO: Measure actual camera mount position on your car and update xyz -->
   <xacro:sensor_d435i parent="${car_name}/base_link" name="camera">
     <origin xyz="0.35 0.0 0.15" rpy="0 0 0"/>
@@ -306,4 +359,7 @@
     </sensor>
   </gazebo>
+  <!-- ================================================================== -->
+  <!-- Ackermann drive plugin                                              -->
+  <!-- ================================================================== -->
   <gazebo>
     <plugin name="gazebo_ros_ackermann_drive" filename="libgazebo_ros_ackermann_drive.so">
@@ -323,10 +379,12 @@
       <wheel_radius>${wheel_radius}</wheel_radius>
       <wheel_diameter>${wheel_radius * 2}</wheel_diameter>
-      <max_steer>0.5</max_steer>
+      <!-- steering limit from VESC servo config -->
+      <max_steer>${max_steering_angle}</max_steer>
       <max_speed>5.0</max_speed>
-      <max_wheel_torque>100.0</max_wheel_torque>
-      <linear_velocity_pid_gain>5.0 0.5 0.05</linear_velocity_pid_gain>
-      <left_steering_pid_gain>25.0 2.0 0.3</left_steering_pid_gain>
-      <right_steering_pid_gain>25.0 2.0 0.3</right_steering_pid_gain>
+      <max_wheel_torque>20.0</max_wheel_torque>
+      <!-- PID gains -->
+      <linear_velocity_pid_gain>3.0 0.3 0.03</linear_velocity_pid_gain>
+      <left_steering_pid_gain>12.0 1.0 0.15</left_steering_pid_gain>
+      <right_steering_pid_gain>12.0 1.0 0.15</right_steering_pid_gain>
       <publish_odom>true</publish_odom>
       <publish_odom_tf>true</publish_odom_tf>
