Commit message: chore: updated f1tenth xacro file

File: urdf/f1tenth.urdf.xacro (robot description, xacro)
@@ -1,19 +1,19 @@
 <?xml version="1.0"?>
 <!--
-  URDF for F1Tenth Gazebo simulation.
-    - body_mass:  18.0 kg  → 3.5 kg   (realistic 1/10 scale car weight)
-    - wheel_mass: 0.5 kg   → 0.1 kg   (realistic RC tire weight)
-    - hinge_mass: 0.5 kg   → 0.1 kg   (lightweight steering knuckle)
-    - Body inertia recalculated for 3.5 kg solid box
-    - Wheel inertia recalculated for 0.1 kg cylinder
-    - Steering hinge limits: ±0.5 rad → ±0.31 rad (from VESC servo clamp)
-    - Steering hinge velocity: 5.0 → 3.2 rad/s (from throttle_interpolator max_servo_speed)
-    - Tire friction: mu1 1.5→0.8, mu2 2.5→1.0 (indoor smooth surface)
-    - Contact stiffness: kp 500000→100000 (less rigid tire contact)
-    - Laser position: 0.275→0.27 m (matches static_transform_publisher in launch)
-    - max_steer: 0.5→0.31 rad (matches VESC-derived steering limit)
-    - max_wheel_torque: 100→20 Nm (matches 2.5 m/s² accel limit at 3.5 kg)
-    - Steering PID: reduced for lighter mass to prevent overshoot
-    - Velocity PID: reduced for lighter mass
+  Corrected URDF for F1Tenth Gazebo simulation — v2
+  Changes from v1:
+    - body_mass: 3.5 → 5.0 kg (more realistic with all components)
+    - Body inertia recalculated for 5.0 kg
+    - Tire friction increased: mu1 0.8→1.0, mu2 1.0→1.5 (prevent drifting)
+    - Contact softness: kp 100000→50000, kd 10→50 (softer tire contact)
+    - max_wheel_torque: 20→10 Nm (prevent wheelspin / oversteer)
+    - Wheel damping: 0.01→0.05, friction 0.0→0.01 (reduce free spinning)
+    - Hinge damping: 0.1→0.2 (prevent steering oscillation)
+  Original changes from stock (carried over from v1):
+    - Steering limits: ±0.5 → ±0.31 rad (from VESC servo config)
+    - Steering velocity: 5.0 → 3.2 rad/s (from throttle_interpolator)
+    - Laser position: 0.275 → 0.27 m (matches launch file)
+    - max_steer: 0.5 → 0.31 rad
+    - PID gains reduced for realistic mass
 -->
 <robot xmlns:xacro="http://www.ros.org/wiki/xacro" name="racecar">
@@ -28,5 +28,5 @@
   <xacro:property name="wheel_length" value="0.0381" />
   <xacro:property name="car_name" value="ego_racecar" />
-  <!-- laser position from static_transform_publisher: 0.27m forward, 0.11m up -->
+  <!-- Laser: matches static_transform_publisher in launch file -->
   <xacro:property name="laser_distance_from_base_link" value="0.27" />
   <xacro:property name="laser_height" value="0.05" />
@@ -34,29 +34,29 @@
   <!-- ================================================================== -->
   <!-- Mass properties                                                     -->
-  <!--   Real F1Tenth car: ~3.2-3.8 kg total (chassis + battery + compute  -->
-  <!--   + LiDAR + VESC). Using 3.5 kg as body mass.                      -->
-  <!--   RC tires: ~80-120g each. Using 0.1 kg.                           -->
-  <!-- ================================================================== -->
-  <xacro:property name="body_mass" value="3.5" />
-  <xacro:property name="wheel_mass" value="0.1" />
+  <!-- Realistic weight with all components:                               -->
+  <!--   Traxxas Slash 4x4 chassis + motor: ~2.5 kg                       -->
+  <!--   Compute (Jetson/NUC):              ~0.5-0.8 kg                   -->
+  <!--   LiPo battery:                      ~0.3-0.5 kg                   -->
+  <!--   Hokuyo LiDAR + metal riser:        ~0.3 kg                       -->
+  <!--   VESC + RealSense + wiring:         ~0.4 kg                       -->
+  <!--   Mounting plates, brackets, screws:  ~0.5-1.0 kg                  -->
+  <!--   Total: ~4.5-5.5 kg → using 5.0 kg                               -->
+  <!-- ================================================================== -->
+  <xacro:property name="body_mass" value="5.0" />
+  <xacro:property name="wheel_mass" value="0.15" />
   <xacro:property name="hinge_mass" value="0.1" />
-  <!-- Steering limits derived from VESC config                 -->
-  <!--   servo range [0.15, 0.85], gain=-1.2135, offset=0.5304            -->
-  <!--   max angle = (0.85 - 0.5304) / 1.2135 ≈ 0.264 rad               -->
-  <!--   min angle = (0.15 - 0.5304) / 1.2135 ≈ -0.314 rad              -->
-  <!--   Using ±0.31 as symmetric approximation                           -->
+  <!-- Steering limits from VESC servo config -->
   <xacro:property name="max_steering_angle" value="0.31" />
-  <!-- Steering velocity from throttle_interpolator config      -->
   <xacro:property name="max_steering_velocity" value="3.2" />
   <!-- ================================================================== -->
-  <!-- Body inertia at 3.5 kg (solid box: 0.25 x 0.2032 x 0.1)-->
-  <!--   ixx = (1/12)*3.5*(0.2032² + 0.1²)  = 0.0150                     -->
-  <!--   iyy = (1/12)*3.5*(0.25²   + 0.1²)  = 0.0347                     -->
-  <!--   izz = (1/12)*3.5*(0.25²   + 0.2032²)= 0.0439                    -->
-  <!-- ================================================================== -->
-  <!-- ================================================================== -->
-  <!-- Wheel inertia at 0.1 kg (cylinder r=0.0508, h=0.0381)   -->
-  <!--   ixx = iyy = (1/12)*0.1*(3*0.0508² + 0.0381²) = 0.0000766        -->
-  <!--   izz = (1/2)*0.1*0.0508²                       = 0.000129         -->
+  <!-- Body inertia at 5.0 kg (solid box: 0.25 x 0.2032 x 0.1)           -->
+  <!--   ixx = (1/12)*5.0*(0.2032^2 + 0.1^2)   = 0.0215                  -->
+  <!--   iyy = (1/12)*5.0*(0.25^2   + 0.1^2)    = 0.0497                  -->
+  <!--   izz = (1/12)*5.0*(0.25^2   + 0.2032^2) = 0.0627                  -->
+  <!-- ================================================================== -->
+  <!-- ================================================================== -->
+  <!-- Wheel inertia at 0.15 kg (cylinder r=0.0508, h=0.0381)             -->
+  <!--   ixx = iyy = (1/12)*0.15*(3*0.0508^2 + 0.0381^2) = 0.000115      -->
+  <!--   izz = (1/2)*0.15*0.0508^2                        = 0.000194      -->
   <!-- ================================================================== -->
   <!-- ================================================================== -->
@@ -86,11 +86,10 @@
       </geometry>
     </collision>
-    <!-- mass and inertia for 3.5 kg -->
     <inertial>
       <origin xyz="${wheelbase/2} 0 ${ground_offset+height/2}"/>
       <mass value="${body_mass}"/>
-      <inertia ixx="0.0150" ixy="0.0" ixz="0.0"
-               iyy="0.0347" iyz="0.0"
-               izz="0.0439"/>
+      <inertia ixx="0.0215" ixy="0.0" ixz="0.0"
+               iyy="0.0497" iyz="0.0"
+               izz="0.0627"/>
     </inertial>
   </link>
@@ -104,5 +103,4 @@
     <parent link="${car_name}/base_link"/>
     <child link="${car_name}/laser_model"/>
-    <!-- x=0.27 to match static_transform_publisher in launch file -->
     <origin xyz="${laser_distance_from_base_link} 0 ${ground_offset+height+(laser_height/2)}"/>
   </joint>
@@ -124,5 +122,6 @@
     <axis xyz="0 1 0"/>
     <limit effort="100.0" velocity="100.0"/>
-    <dynamics damping="0.01" friction="0.0"/>
+    <!-- Increased damping + friction to prevent free spinning -->
+    <dynamics damping="0.05" friction="0.01"/>
   </joint>
   <link name="${car_name}/back_left_wheel">
@@ -140,20 +139,20 @@
       </geometry>
     </collision>
-    <!-- wheel inertia at 0.1 kg -->
     <inertial>
       <origin rpy="${pi/2} 0 0"/>
       <mass value="${wheel_mass}"/>
-      <inertia ixx="0.0000766" ixy="0.0" ixz="0.0"
-               iyy="0.0000766" iyz="0.0"
-               izz="0.000129"/>
-    </inertial>
-  </link>
-  <!-- tire friction for indoor smooth surface -->
+      <inertia ixx="0.000115" ixy="0.0" ixz="0.0"
+               iyy="0.000115" iyz="0.0"
+               izz="0.000194"/>
+    </inertial>
+  </link>
+  <!-- Tire friction: tuned for treaded RC tires on smooth indoor floor -->
+  <!-- Higher mu prevents drifting; softer kp/kd gives realistic contact -->
   <gazebo reference="${car_name}/back_left_wheel">
     <material>Gazebo/Black</material>
-    <mu1>0.8</mu1>
-    <mu2>1.0</mu2>
-    <kp>100000.0</kp>
-    <kd>10.0</kd>
+    <mu1>1.0</mu1>
+    <mu2>1.5</mu2>
+    <kp>50000.0</kp>
+    <kd>50.0</kd>
     <minDepth>0.001</minDepth>
   </gazebo>
@@ -167,5 +166,5 @@
     <axis xyz="0 1 0"/>
     <limit effort="100.0" velocity="100.0"/>
-    <dynamics damping="0.01" friction="0.0"/>
+    <dynamics damping="0.05" friction="0.01"/>
   </joint>
   <link name="${car_name}/back_right_wheel">
@@ -183,20 +182,18 @@
       </geometry>
     </collision>
-    <!-- wheel inertia at 0.1 kg -->
     <inertial>
       <origin rpy="${pi/2} 0 0"/>
       <mass value="${wheel_mass}"/>
-      <inertia ixx="0.0000766" ixy="0.0" ixz="0.0"
-               iyy="0.0000766" iyz="0.0"
-               izz="0.000129"/>
-    </inertial>
-  </link>
-  <!-- tire friction for indoor smooth surface -->
+      <inertia ixx="0.000115" ixy="0.0" ixz="0.0"
+               iyy="0.000115" iyz="0.0"
+               izz="0.000194"/>
+    </inertial>
+  </link>
   <gazebo reference="${car_name}/back_right_wheel">
     <material>Gazebo/Black</material>
-    <mu1>0.8</mu1>
-    <mu2>1.0</mu2>
-    <kp>100000.0</kp>
-    <kd>10.0</kd>
+    <mu1>1.0</mu1>
+    <mu2>1.5</mu2>
+    <kp>50000.0</kp>
+    <kd>50.0</kd>
     <minDepth>0.001</minDepth>
   </gazebo>
@@ -204,5 +201,4 @@
   <!-- Front left steering hinge + wheel                                   -->
   <!-- ================================================================== -->
-  <!-- steering limits from VESC servo config, velocity from throttle_interpolator -->
   <joint name="base_to_front_left_hinge" type="revolute">
     <parent link="${car_name}/base_link"/>
@@ -211,5 +207,6 @@
     <axis xyz="0 0 1"/>
     <limit lower="-${max_steering_angle}" upper="${max_steering_angle}" effort="10.0" velocity="${max_steering_velocity}"/>
-    <dynamics damping="0.1" friction="0.0"/>
+    <!-- Higher damping prevents steering oscillation at lighter mass -->
+    <dynamics damping="0.2" friction="0.01"/>
   </joint>
   <link name="${car_name}/front_left_hinge">
@@ -226,5 +223,5 @@
     <axis xyz="0 1 0"/>
     <limit effort="100.0" velocity="100.0"/>
-    <dynamics damping="0.01" friction="0.0"/>
+    <dynamics damping="0.05" friction="0.01"/>
   </joint>
   <link name="${car_name}/front_left_wheel">
@@ -242,20 +239,18 @@
       </geometry>
     </collision>
-    <!-- wheel inertia at 0.1 kg -->
     <inertial>
       <origin rpy="${pi/2} 0 0"/>
       <mass value="${wheel_mass}"/>
-      <inertia ixx="0.0000766" ixy="0.0" ixz="0.0"
-               iyy="0.0000766" iyz="0.0"
-               izz="0.000129"/>
-    </inertial>
-  </link>
-  <!-- tire friction for indoor smooth surface -->
+      <inertia ixx="0.000115" ixy="0.0" ixz="0.0"
+               iyy="0.000115" iyz="0.0"
+               izz="0.000194"/>
+    </inertial>
+  </link>
   <gazebo reference="${car_name}/front_left_wheel">
     <material>Gazebo/Black</material>
-    <mu1>0.8</mu1>
-    <mu2>1.0</mu2>
-    <kp>100000.0</kp>
-    <kd>10.0</kd>
+    <mu1>1.0</mu1>
+    <mu2>1.5</mu2>
+    <kp>50000.0</kp>
+    <kd>50.0</kd>
     <minDepth>0.001</minDepth>
   </gazebo>
@@ -263,5 +258,4 @@
   <!-- Front right steering hinge + wheel                                  -->
   <!-- ================================================================== -->
-  <!-- steering limits from VESC servo config, velocity from throttle_interpolator -->
   <joint name="base_to_front_right_hinge" type="revolute">
     <parent link="${car_name}/base_link"/>
@@ -270,5 +264,5 @@
     <axis xyz="0 0 1"/>
     <limit lower="-${max_steering_angle}" upper="${max_steering_angle}" effort="10.0" velocity="${max_steering_velocity}"/>
-    <dynamics damping="0.1" friction="0.0"/>
+    <dynamics damping="0.2" friction="0.01"/>
   </joint>
   <link name="${car_name}/front_right_hinge">
@@ -285,5 +279,5 @@
     <axis xyz="0 1 0"/>
     <limit effort="100.0" velocity="100.0"/>
-    <dynamics damping="0.01" friction="0.0"/>
+    <dynamics damping="0.05" friction="0.01"/>
   </joint>
   <link name="${car_name}/front_right_wheel">
@@ -301,27 +295,26 @@
       </geometry>
     </collision>
-    <!-- wheel inertia at 0.1 kg -->
     <inertial>
       <origin rpy="${pi/2} 0 0"/>
       <mass value="${wheel_mass}"/>
-      <inertia ixx="0.0000766" ixy="0.0" ixz="0.0"
-               iyy="0.0000766" iyz="0.0"
-               izz="0.000129"/>
-    </inertial>
-  </link>
-  <!-- tire friction for indoor smooth surface -->
+      <inertia ixx="0.000115" ixy="0.0" ixz="0.0"
+               iyy="0.000115" iyz="0.0"
+               izz="0.000194"/>
+    </inertial>
+  </link>
   <gazebo reference="${car_name}/front_right_wheel">
     <material>Gazebo/Black</material>
-    <mu1>0.6</mu1>
-    <mu2>0.8</mu2>
-    <kp>100000.0</kp>
-    <kd>10.0</kd>
+    <mu1>1.0</mu1>
+    <mu2>1.5</mu2>
+    <kp>50000.0</kp>
+    <kd>50.0</kd>
     <minDepth>0.001</minDepth>
   </gazebo>
   <!-- ================================================================== -->
   <!-- Intel RealSense D435i Camera                                        -->
+  <!-- NOTE: Requires ros-foxy-realsense2-description to be installed.     -->
+  <!-- Comment out the next two blocks if not available.                    -->
   <!-- ================================================================== -->
   <xacro:include filename="$(find realsense2_description)/urdf/_d435i.urdf.xacro" />
-  <!-- TODO: Measure actual camera mount position on your car and update xyz -->
   <xacro:sensor_d435i parent="${car_name}/base_link" name="camera">
     <origin xyz="0.35 0.0 0.15" rpy="0 0 0"/>
@@ -379,12 +372,14 @@
       <wheel_radius>${wheel_radius}</wheel_radius>
       <wheel_diameter>${wheel_radius * 2}</wheel_diameter>
-      <!-- steering limit from VESC servo config -->
       <max_steer>${max_steering_angle}</max_steer>
       <max_speed>5.0</max_speed>
-      <max_wheel_torque>20.0</max_wheel_torque>
-      <!-- PID gains -->
-      <linear_velocity_pid_gain>3.0 0.3 0.03</linear_velocity_pid_gain>
-      <left_steering_pid_gain>12.0 1.0 0.15</left_steering_pid_gain>
-      <right_steering_pid_gain>12.0 1.0 0.15</right_steering_pid_gain>
+      <!-- Reduced torque: prevents wheelspin and oversteer -->
+      <!-- At 5 kg, 10 Nm on 0.05m wheels = ~40 m/s^2 theoretical max -->
+      <!-- Actual acceleration limited by friction to ~2-3 m/s^2 -->
+      <max_wheel_torque>10.0</max_wheel_torque>
+      <!-- PID gains tuned for 5 kg mass -->
+      <linear_velocity_pid_gain>4.0 0.4 0.04</linear_velocity_pid_gain>
+      <left_steering_pid_gain>15.0 1.5 0.2</left_steering_pid_gain>
+      <right_steering_pid_gain>15.0 1.5 0.2</right_steering_pid_gain>
       <publish_odom>true</publish_odom>
       <publish_odom_tf>true</publish_odom_tf>

Commit message: using rectangular map

File: urdf/f1tenth.urdf.xacro (robot description, xacro)
@@ -21,5 +21,5 @@
   <!-- Geometric properties                                                -->
   <!-- ================================================================== -->
-  <xacro:property name="wheelbase" value="0.25" />
+  <xacro:property name="wheelbase" value="0.2" />
   <xacro:property name="width" value="0.2032" />
   <xacro:property name="height" value="0.1" />
@@ -47,5 +47,5 @@
   <xacro:property name="hinge_mass" value="0.1" />
   <!-- Steering limits from VESC servo config -->
-  <xacro:property name="max_steering_angle" value="0.31" />
+  <xacro:property name="max_steering_angle" value="0.7" />
   <xacro:property name="max_steering_velocity" value="3.2" />
   <!-- ================================================================== -->
@@ -105,4 +105,26 @@
     <origin xyz="${laser_distance_from_base_link} 0 ${ground_offset+height+(laser_height/2)}"/>
   </joint>
+  <gazebo reference="${car_name}/base_link">
+    <sensor name="imu" type="imu">
+        <always_on>true</always_on>
+        <update_rate>200</update_rate>
+        <imu>
+            <angular_velocity>
+                <x><noise type="gaussian"><mean>0</mean><stddev>0.001</stddev></noise></x>
+                <y><noise type="gaussian"><mean>0</mean><stddev>0.001</stddev></noise></y>
+                <z><noise type="gaussian"><mean>0</mean><stddev>0.001</stddev></noise></z>
+            </angular_velocity>
+            <linear_acceleration>
+                <x><noise type="gaussian"><mean>0</mean><stddev>0.01</stddev></noise></x>
+                <y><noise type="gaussian"><mean>0</mean><stddev>0.01</stddev></noise></y>
+                <z><noise type="gaussian"><mean>0</mean><stddev>0.01</stddev></noise></z>
+            </linear_acceleration>
+        </imu>
+        <plugin name="imu_plugin" filename="libgazebo_ros_imu_sensor.so">
+            <ros><remapping>~/out:=/imu</remapping></ros>
+            <frame_name>${car_name}/base_link</frame_name>
+        </plugin>
+    </sensor>
+  </gazebo>
   <link name="${car_name}/laser_model">
     <visual>
@@ -112,5 +134,50 @@
       <material name="black"/>
     </visual>
-  </link>
+    <!-- <collision>
+      <geometry>
+        <cylinder radius="${laser_radius}" length="${laser_height}"/>
+      </geometry>
+    </collision>
+    <inertial>
+      <mass value="0.13"/>
+      <inertia ixx="0.0001" ixy="0.0" ixz="0.0"
+               iyy="0.0001" iyz="0.0"
+               izz="0.0001"/>
+    </inertial> -->
+  </link>
+  <gazebo reference="${car_name}/laser_model">
+    <sensor name="lidar" type="ray">
+      <always_on>true</always_on>
+      <visualize>false</visualize>
+      <update_rate>20</update_rate>
+      <ray>
+        <scan>
+          <horizontal>
+            <samples>1080</samples>
+            <resolution>1</resolution>
+            <min_angle>-2.35</min_angle>
+            <max_angle>2.35</max_angle>
+          </horizontal>
+        </scan>
+        <range>
+          <min>0.1</min>
+          <max>30.0</max>
+          <resolution>0.01</resolution>
+        </range>
+        <noise>
+          <type>gaussian</type>
+          <mean>0.0</mean>
+          <stddev>0.01</stddev>
+        </noise>
+      </ray>
+      <plugin name="scan" filename="libgazebo_ros_ray_sensor.so">
+        <ros>
+          <remapping>~/out:=/scan</remapping>
+        </ros>
+        <output_type>sensor_msgs/LaserScan</output_type>
+        <frame_name>${car_name}/laser_model</frame_name>
+      </plugin>
+    </sensor>
+  </gazebo>
   <!-- ================================================================== -->
   <!-- Back left wheel                                                     -->
@@ -151,6 +218,6 @@
   <gazebo reference="${car_name}/back_left_wheel">
     <material>Gazebo/Black</material>
-    <mu1>1.0</mu1>
-    <mu2>1.5</mu2>
+    <mu1>2.0</mu1>
+    <mu2>2.0</mu2>
     <kp>50000.0</kp>
     <kd>50.0</kd>
@@ -192,6 +259,6 @@
   <gazebo reference="${car_name}/back_right_wheel">
     <material>Gazebo/Black</material>
-    <mu1>1.0</mu1>
-    <mu2>1.5</mu2>
+    <mu1>2.0</mu1>
+    <mu2>2.0</mu2>
     <kp>50000.0</kp>
     <kd>50.0</kd>
@@ -249,6 +316,6 @@
   <gazebo reference="${car_name}/front_left_wheel">
     <material>Gazebo/Black</material>
-    <mu1>1.0</mu1>
-    <mu2>1.5</mu2>
+    <mu1>2.0</mu1>
+    <mu2>2.0</mu2>
     <kp>50000.0</kp>
     <kd>50.0</kd>
@@ -305,6 +372,6 @@
   <gazebo reference="${car_name}/front_right_wheel">
     <material>Gazebo/Black</material>
-    <mu1>1.0</mu1>
-    <mu2>1.5</mu2>
+    <mu1>2.0</mu1>
+    <mu2>2.0</mu2>
     <kp>50000.0</kp>
     <kd>50.0</kd>
@@ -361,5 +428,5 @@
         <remapping>odom:=odom</remapping>
       </ros>
-      <update_rate>50.0</update_rate>
+      <update_rate>100.0</update_rate>
       <left_steering_joint>base_to_front_left_hinge</left_steering_joint>
       <right_steering_joint>base_to_front_right_hinge</right_steering_joint>
@@ -383,6 +450,6 @@
       <right_steering_pid_gain>15.0 1.5 0.2</right_steering_pid_gain>
       <publish_odom>true</publish_odom>
-      <publish_odom_tf>true</publish_odom_tf>
-      <publish_wheel_tf>true</publish_wheel_tf>
+      <publish_odom_tf>false</publish_odom_tf>
+      <publish_wheel_tf>false</publish_wheel_tf>
       <odometry_frame>odom</odometry_frame>
       <robot_base_frame>${car_name}/base_link</robot_base_frame>
